File: hardware/KiCAD/WS2812B.kicad_sch (KiCad schematic)
At the start: 2 parts, among them U11 74AHCT1G125

Commit message: update
Parts:
- R70: value 330Ω/0603 -> 330Ω; DigiKey_Part_Number (none) -> 541-330HCT-ND; Manufacturer_Name (none) -> CRCW0603330RFKEA; Manufacturer_Part_Number (none) -> Vishay Dale; PACKAGE (none) -> 0603; Part name RCS0603330RFKEA -> (none); Power (none) -> 0.125W, 1/8W; Tolerance (none) -> 1%
- U11: DigiKey_Part_Number (none) -> 296-4709-1-ND; Manufacturer_Name (none) -> SN74AHCT1G125DCKR; Manufacturer_Part_Number (none) -> Texas Instruments; PACKAGE (none) -> 5-TSSOP, SC-70-5, SOT-353; Part name SN74AHCT1G125DCKR -> (none)
Changed lines of the file:
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@@
 			)
 		)
-		(property "Part name" "SN74AHCT1G125DCKR"
-			(at 156.21 86.36 0)
-			(effects
-				(font
-					(size 0.762 0.762)
-				)
-				(hide yes)
-			)
-		)
-		(property "DigiKey_Part_Number" ""
+		(property "DigiKey_Part_Number" "296-4709-1-ND"
 			(at 156.21 86.36 0)
 			(effects
@@
 		)
 		(property "Tolerance" ""
+			(at 156.21 86.36 0)
+			(effects
+				(font
+					(size 1.27 1.27)
+				)
+				(hide yes)
+			)
+		)
+		(property "Manufacturer_Name" "SN74AHCT1G125DCKR"
+			(at 156.21 86.36 0)
+			(effects
+				(font
+					(size 1.27 1.27)
+				)
+				(hide yes)
+			)
+		)
+		(property "Manufacturer_Part_Number" "Texas Instruments"
+			(at 156.21 86.36 0)
+			(effects
+				(font
+					(size 1.27 1.27)
+				)
+				(hide yes)
+			)
+		)
+		(property "PACKAGE" "5-TSSOP, SC-70-5, SOT-353"
+			(at 156.21 86.36 0)
+			(effects
+				(font
+					(size 1.27 1.27)
+				)
+				(hide yes)
+			)
+		)
+		(property "MPN" ""
+			(at 156.21 86.36 0)
+			(effects
+				(font
+					(size 1.27 1.27)
+				)
+				(hide yes)
+			)
+		)
+		(property "OC_FARNELL" ""
+			(at 156.21 86.36 0)
+			(effects
+				(font
+					(size 1.27 1.27)
+				)
+				(hide yes)
+			)
+		)
+		(property "OC_NEWARK" ""
+			(at 156.21 86.36 0)
+			(effects
+				(font
+					(size 1.27 1.27)
+				)
+				(hide yes)
+			)
+		)
+		(property "SUPPLIER" ""
 			(at 156.21 86.36 0)
 			(effects
@@
 			)
 		)
-		(property "Value" "330Ω/0603"
+		(property "Value" "330Ω"
 			(at 174.752 84.582 90)
 			(effects
@@
 			)
 		)
-		(property "Part name" "RCS0603330RFKEA"
-			(at 171.45 86.36 0)
-			(effects
-				(font
-					(size 0.762 0.762)
-				)
-				(hide yes)
-			)
-		)
-		(property "DigiKey_Part_Number" ""
+		(property "DigiKey_Part_Number" "541-330HCT-ND"
 			(at 171.45 86.36 90)
 			(effects
@@
 			)
 		)
-		(property "Power" ""
-			(at 171.45 86.36 90)
-			(effects
-				(font
-					(size 1.27 1.27)
-				)
-				(hide yes)
-			)
-		)
-		(property "Tolerance" ""
-			(at 171.45 86.36 90)
-			(effects
+		(property "Power" "0.125W, 1/8W"
+			(at 171.45 86.36 90)
+			(effects
+				(font
+					(size 1.27 1.27)
+				)
+				(hide yes)
+			)
+		)
+		(property "Tolerance" "1%"
+			(at 171.45 86.36 90)
+			(effects
+				(font
+					(size 1.27 1.27)
+				)
+				(hide yes)
+			)
+		)
+		(property "Manufacturer_Name" "CRCW0603330RFKEA"
+			(at 171.45 86.36 90)
+			(effects
+				(font
+					(size 1.27 1.27)
+				)
+				(hide yes)
+			)
+		)
+		(property "Manufacturer_Part_Number" "Vishay Dale"
+			(at 171.45 86.36 90)
+			(effects
+				(font
+					(size 1.27 1.27)
+				)
+				(hide yes)
+			)
+		)
+		(property "PACKAGE" "0603"
+			(at 171.45 86.36 90)
+			(effects
+				(font
+					(size 1.27 1.27)
+				)
+				(hide yes)
+			)
+		)
+		(property "MPN" ""
+			(at 171.45 86.36 90)
+			(effects
+				(font
+					(size 1.27 1.27)
+				)
+				(hide yes)
+			)
+		)
+		(property "OC_FARNELL" ""
+			(at 171.45 86.36 90)
+			(effects
+				(font
+					(size 1.27 1.27)
+				)
+				(hide yes)
+			)
+		)
+		(property "OC_NEWARK" ""
+			(at 171.45 86.36 90)
+			(effects
+				(font
+					(size 1.27 1.27)
+				)
+				(hide yes)
+			)
+		)
+		(property "SUPPLIER" ""
+			(at 171.45 86.36 90)
+			(effects

Commit message: update
Other:
- title: Czujnik parametrów środowiskowych -> Enviromental parameters multi-sensor
Changed lines of the file:
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@@
 	(paper "A4")
 	(title_block
-		(title "Czujnik parametrów środowiskowych")
+		(title "Enviromental parameters multi-sensor")
 		(date "2026-01-20")
 		(rev "1.0")
