File: hardware/KiCAD/pow_supply.kicad_sch (KiCad schematic)
At the start: 18 parts, among them U8 TPS563208DDCR, U9 TPS563208DDCR

Commit message: update
Parts:
- R56: value 56,2kΩ/0603 -> 56,2kΩ; DigiKey_Part_Number (none) -> 541-56.2KHCT-ND; Manufacturer_Name (none) -> CRCW060356K2FKEA; Manufacturer_Part_Number (none) -> Vishay Dale; PACKAGE (none) -> 0805; Part name RCS060356K2FKEA -> (none); Power (none) -> 0.25W, 1/4W; Tolerance (none) -> 1%
- R58: value 33,2kΩ/0603 -> 33,2kΩ; DigiKey_Part_Number (none) -> 541-33.2KHCT-ND; Manufacturer_Name (none) -> CRCW060333K2FKEA; Manufacturer_Part_Number (none) -> Vishay Dale; PACKAGE (none) -> 0805; Part name RCS060333K2FKEA -> (none); Power (none) -> 0.25W, 1/4W; Tolerance (none) -> 1%
- U8, U9: value TPS563208DDCR -> TPS563208; DigiKey_Part_Number (none) -> 296-44844-1-ND; Manufacturer_Name (none) -> TPS563208DDCR; Manufacturer_Part_Number (none) -> Texas Instruments; PACKAGE (none) -> SOT-23-6 Thin, TSOT-23-6; Part name TPS563208DDCR -> (none)

Commit message: update
Other:
- title: Czujnik parametrów środowiskowych -> Enviromental parameters multi-sensor
Changed lines of the file:
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@@
 	(paper "A4")
 	(title_block
-		(title "Czujnik parametrów środowiskowych")
+		(title "Enviromental parameters multi-sensor")
 		(date "2026-01-20")
 		(rev "1.0")
