File: hardware/KiCAD/usb_uart.kicad_sch (KiCad schematic)
At the start: 14 parts, among them Q1 BC846B, U2 CP2102N-A02-GQFN24R

Commit message: update
Parts:
- U2: value CP2102N-A02-GQFN24R -> CP2102N; DigiKey_Part_Number (none) -> 336-5888-1-ND; Manufacturer_Name (none) -> CP2102N-A02-GQFN24R; Manufacturer_Part_Number (none) -> Silicon Labs; PACKAGE (none) -> 24-QFN; Part name CP2102N-A02-GQFN24R -> (none)

Commit message: update
Other:
- title: Czujnik parametrów środowiskowych -> Enviromental parameters multi-sensor
Changed lines of the file:
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@@
 	(paper "A4")
 	(title_block
-		(title "Czujnik parametrów środowiskowych")
+		(title "Enviromental parameters multi-sensor")
 		(date "2026-01-20")
 		(rev "1.0")
