File: hardware/KiCAD/mpair.kicad_pcb (KiCad board)
At the start: 2 copper layers, 100 x 100 mm, 195 parts, among them J3 DX07S016JA1R1500, J4 ARJP11A-MASA-B-A-EMU2, K1 G6K-2G-TR DC5, Q1 BC846B, Q2 FDMC2523P, Q3 FDS86242, Q4 CSD19534Q, Q5 FCX493, Q6 FCX493, Q7 CSD19534Q, Q8 MMBT3904, T1 PA4065NL, U1 USBLC6-2SC6, U10 ESP32-C6-WROOM-1U, U11 74AHCT1G125, U2 CP2102N, U3 ESDS314, U4 W5500, U5 TPS23754, U6 HMHA2801A, U7 PC357N, U8 TPS563208, U9 TPS563208, Y1 ECS-2520MV-250

Commit message: update
Parts:
- C1: moved to B.Cu
- moved C1 17.8 mm to (28.2, 64.2), turned to -90 degrees
- moved C4 8.78 mm to (37.0, 64.2), turned to -90 degrees
- moved L2 8.08 mm to (35.9, 70.2)
- moved L1 5.70 mm to (35.9, 58.5)
- moved D2 5.64 mm to (41.8, 61.5), turned to 90 degrees
- moved J4 0.60 mm to (40.0, 78.2)
- moved C3 0.56 mm to (31.0, 84.0)
- moved R1 0.50 mm to (27.0, 84.0)
Routing:
- net Net-(C3-Pad1): track 14.4 -> 0.00 mm
- net SHIELD: track 13.0 -> 0.00 mm

Commit message: update
Parts:
- C18, C2, C20, R18, U3: moved to B.Cu
- J1, J2: value ~ -> PJ-063AH; footprint MarPi82:PJ-002AH-SMT-TR -> Connector_BarrelJack:BarrelJack_CUI_PJ-063AH_Horizontal_CircularHoles
- moved U3 188.6 mm to (38.7, 22.1)
- moved R12 185.5 mm to (28.2, 19.9)
- moved RN1 176.9 mm to (51.5, 24.9)
- moved R20 173.0 mm to (44.7, 20.4)
- moved R14 171.8 mm to (43.7, 24.5), turned to -90 degrees
- moved R19 171.2 mm to (44.7, 22.1)
- moved D3 171.0 mm to (54.2, 23.3), turned to -90 degrees
- moved D4 170.7 mm to (54.2, 26.4), turned to 90 degrees
- moved C18 168.8 mm to (60.4, 26.4), turned to 180 degrees
- moved R13 167.3 mm to (47.5, 24.5), turned to -90 degrees
- moved R16 166.5 mm to (45.6, 24.5), turned to -90 degrees
- moved R15 166.4 mm to (47.1, 32.2), turned to 90 degrees
- moved R21 165.2 mm to (50.7, 28.4), turned to -90 degrees
- moved R17 164.4 mm to (47.1, 28.7), turned to -90 degrees
- moved U4 163.7 mm to (61.4, 26.4)
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Connections:
- C11 pad 1: /Interface PHY/RD+ -> /Interface PHY/RD-
- C12 pad 1: /Interface PHY/RD- -> /Interface PHY/RD+
- R14 pad 2: /Interface PHY/TD- -> /Interface PHY/TD+
- R16 pad 2: /Interface PHY/TD+ -> /Interface PHY/TD-
- RN1 pad 1: /Interface PHY/TD+ -> /Interface PHY/TD-
- RN1 pad 2: /Interface PHY/TD- -> /Interface PHY/TD+
- U3 pad 4: /Interface PHY/TD+ -> /Interface PHY/TD-
- U3 pad 5: /Interface PHY/TD- -> /Interface PHY/TD+
- U4 pad 1: Net-(D3-A2) -> Net-(D3-A1)
- U4 pad 2: Net-(D3-A1) -> Net-(D3-A2)
- U4 pad 5: Net-(D4-A1) -> Net-(D4-A2)
- U4 pad 6: Net-(D4-A2) -> Net-(D4-A1)
Routing:
- net +3V3_PHY: track 0.00 -> 62.5 mm, vias 0 -> 3
- net SHIELD: track 0.00 -> 59.2 mm
- net +3V3_PHY_A: track 0.00 -> 43.0 mm, vias 0 -> 4
- net AGND: track 0.00 -> 36.0 mm
- net Net-(U4-LINKLED): track 0.00 -> 32.7 mm, vias 0 -> 2
- net Net-(U4-ACTLED): track 0.00 -> 31.6 mm, vias 0 -> 2
- net /Interface PHY/LED_LNK: track 0.00 -> 30.4 mm
- net GND: track 0.00 -> 26.9 mm, vias 0 -> 4
- net /PoE+ power supply/POE+: track 0.00 -> 23.5 mm
- net /PoE+ power supply/AUXGND: track 0.00 -> 21.9 mm, vias 0 -> 1
- net /Interface PHY/TD-: track 0.00 -> 20.4 mm, vias 0 -> 2
- net /Interface PHY/LED_ACT: track 0.00 -> 19.9 mm
- net Net-(C2-Pad2): track 0.00 -> 18.7 mm
- net Net-(C1-Pad2): track 0.00 -> 18.7 mm
- net /Interface PHY/LED+: track 0.00 -> 18.5 mm
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- added copper zone on B.Cu, net GND
- added copper zone on F.Cu, net GND
- added copper zone on B.Cu, net SHIELD
Other:
- board size 100 x 100 mm -> 100 x 102 mm

Commit message: update
Parts:
- moved C9 161.2 mm to (70.8, 34.1)
- moved Y1 160.6 mm to (71.7, 27.7), turned to 90 degrees
- moved C13 154.1 mm to (69.1, 27.7), turned to 90 degrees
- moved R31 151.9 mm to (69.9, 30.0), turned to 180 degrees
- moved L6 146.7 mm to (66.5, 33.4)
- moved L7 144.6 mm to (66.8, 31.6)
- moved C23 140.7 mm to (69.9, 31.6)
- moved U5 127.0 mm to (55.5, 45.6), turned to -90 degrees
- moved C24 26.8 mm to (49.1, 36.5), turned to 90 degrees
- moved D5 22.2 mm to (45.6, 45.6), turned to -90 degrees
- moved L8 17.7 mm to (45.6, 36.5), turned to 90 degrees
- moved R32 10.5 mm to (39.5, 52.0)
Routing:
- net /PoE+ power supply/VSS: track 0.00 -> 17.3 mm
- net GND: track 26.9 -> 41.7 mm, vias 4 -> 5
- net +3V3_PHY: track 62.5 -> 75.4 mm
- net /PoE+ power supply/POE+: track 23.5 -> 11.7 mm
- net /PoE+ power supply/VDD: track 0.00 -> 8.59 mm
- net +3.3V: track 0.00 -> 5.13 mm
- net /PoE+ power supply/AUXGND: track 21.9 -> 26.3 mm, vias 1 -> 2
- net Net-(U4-XI/CLKIN): track 4.01 -> 8.37 mm
- net +3V3_PHY_A: track 43.0 -> 46.5 mm
- net Net-(U4-ACTLED): track 31.6 -> 34.2 mm
- net Net-(U4-MISO): track 3.60 -> 5.77 mm
- net Net-(U4-SCLK): track 3.66 -> 5.73 mm
- net Net-(U4-~{SCS}): track 3.82 -> 5.69 mm
- net /ESP32-C6/~{RST}_{PHY}: track 4.25 -> 6.02 mm
- net Net-(U4-~{INT}): track 4.13 -> 5.86 mm
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- added copper zone on F.Cu, net /PoE+ power supply/VSS
- added copper zone on F.Cu, net AGND

Commit message: update
Parts:
- moved R34 104.1 mm to (51.2, 36.5), turned to 90 degrees
- moved R36 103.1 mm to (53.1, 36.5), turned to 90 degrees
- moved R33 100.0 mm to (55.0, 36.5), turned to 90 degrees
- moved R35 97.0 mm to (58.8, 36.5), turned to 90 degrees
- moved R37 96.2 mm to (60.6, 36.5), turned to 90 degrees
- moved R38 95.0 mm to (62.6, 36.5), turned to -90 degrees
- moved R32 23.3 mm to (56.9, 36.5), turned to -90 degrees
- moved U5 3.04 mm to (53.5, 43.4), turned to 90 degrees
Routing:
- net Net-(U5-DEN): track 0.00 -> 9.23 mm
- net Net-(U5-CLS): track 0.00 -> 8.55 mm
- net Net-(U5-DT): track 0.00 -> 7.36 mm
- net Net-(U5-APD): track 0.00 -> 6.15 mm
- net Net-(U5-BLNK): track 0.00 -> 3.65 mm
- net Net-(U5-FRS): track 0.00 -> 3.12 mm
- net PGND: track 0.00 -> 0.74 mm
- added copper zone on B.Cu, net PGND

Commit message: update
Parts:
- U7: footprint Package_SO:SOIC-4_4.55x3.7mm_P2.54mm -> Package_SO:OnSemi_751EP_SOIC-4_3.9x4.725mm_P2.54mm
- moved U7 121.0 mm to (49.3, 61.9), turned to -90 degrees
- moved U6 113.2 mm to (55.8, 73.1), turned to 90 degrees
- moved R47 95.8 mm to (62.4, 66.1)
- moved R41 95.7 mm to (62.6, 55.1)
- moved R46 95.6 mm to (62.5, 62.6)
- moved R42 95.4 mm to (62.9, 58.5)
- moved C29 92.8 mm to (57.7, 57.7)
- moved C30 92.8 mm to (57.7, 60.2)
- moved C31 92.8 mm to (57.7, 62.7)
- moved D6 83.1 mm to (60.2, 43.3), turned to -90 degrees
Routing:
- net /PoE+ power supply/AUX: track 13.2 -> 48.1 mm, vias 0 -> 1
- net /PoE+ power supply/VDD: track 8.59 -> 33.8 mm, vias 0 -> 2
- net /PoE+ power supply/VSS: track 17.3 -> 0.14 mm
- net PGND: track 0.74 -> 17.9 mm, vias 0 -> 5
- net Net-(U5-T2P): track 0.00 -> 11.9 mm, vias 0 -> 2

Commit message: update
Parts:
- removed D9: MMBD4148, Package_TO_SOT_SMD:SC-59
- D8: value MMBD4148 -> MMBD4148CC
- moved C36 140.4 mm to (43.6, 84.6), turned to 90 degrees
- moved C27 134.8 mm to (42.7, 54.5)
- moved L9 134.2 mm to (42.7, 63.5)
- moved D12 132.1 mm to (46.4, 88.8)
- moved D11 131.9 mm to (46.8, 84.6)
- moved R45 128.5 mm to (50.9, 59.7)
- moved Q5 128.2 mm to (54.4, 91.8), turned to 90 degrees
- moved R48 127.7 mm to (39.5, 84.7), turned to -90 degrees
- moved R53 126.6 mm to (39.5, 88.1), turned to 90 degrees
- moved R55 126.2 mm to (39.5, 91.5), turned to -90 degrees
- moved R5 125.8 mm to (97.7, 110.2)
- moved R49 125.2 mm to (41.4, 84.7), turned to -90 degrees
- moved R54 125.0 mm to (41.4, 91.5), turned to -90 degrees
- moved R52 124.6 mm to (43.3, 91.5), turned to -90 degrees
- moved C25 122.8 mm to (58.2, 56.5), turned to 90 degrees
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Connections:
- net Net-(C26-Pad1) renamed /PoE+ power supply/Q3D
- net Net-(C26-Pad2) renamed /PoE+ power supply/Q2D
- net Net-(U5-CTL) renamed /PoE+ power supply/CTL
- net Net-(U5-GAT2) renamed /PoE+ power supply/GATE2
- net Net-(U5-T2P) renamed /PoE+ power supply/T2P
- net Net-(U5-VB) renamed /PoE+ power supply/VB
- net Net-(U5-VC) renamed /PoE+ power supply/VC
- C28 pad 2: Net-(D9-A) -> Net-(D8-A2)
- C38 pad 1: Net-(D14-K) -> /PoE+ power supply/V-
- C4 pad 1: +12V -> Net-(D2-A)
- C44 pad 2: /Power supply/+12V -> +12V
- C45 pad 2: /Power supply/+12V -> +12V
- C46 pad 2: /Power supply/+12V -> +12V
- C47 pad 2: /Power supply/+12V -> +12V
- D10 pad 1: Net-(D10-K) -> Net-(D10-A)
- D10 pad 2: Net-(D10-A) -> unconnected-(D10-NC-Pad2)
- D10 pad 3: (no net) -> /PoE+ power supply/V+
- D14 pad 1: Net-(D14-K) -> Net-(D14-A)
- D14 pad 2: Net-(D14-A) -> unconnected-(D14-NC-Pad2)
- D14 pad 3: (no net) -> /PoE+ power supply/V-
- D2 pad 1: /Power supply/+12V -> +12V
- D2 pad 2: +12V -> Net-(D2-A)
- D7 pad 1: PGND -> Net-(D7-A)
- D7 pad 2: Net-(D7-A) -> unconnected-(D7-NC-Pad2)
- D7 pad 3: (no net) -> PGND
- D8 pad 1: Net-(D8-K) -> Net-(D8-A1)
- D8 pad 2: Net-(D8-A) -> Net-(D8-A2)
- D8 pad 3: (no net) -> Net-(D8-K)
- L1 pad 2: +12V -> Net-(D2-A)
- L11 pad 1: Net-(D10-K) -> /PoE+ power supply/V+
- Q4 pad D: Net-(D14-K) -> /PoE+ power supply/V-
- Q5 pad 2: Net-(D10-K) -> /PoE+ power supply/V+
- Q6 pad 2: Net-(D14-K) -> /PoE+ power supply/V-
- Q7 pad D: Net-(D10-K) -> /PoE+ power supply/V+
- R50 pad 1: Net-(D10-K) -> /PoE+ power supply/V+
- R51 pad 1: Net-(D14-K) -> /PoE+ power supply/V-
- T1 pad 10: Net-(D14-K) -> /PoE+ power supply/V-
- T1 pad 4: Net-(D8-A) -> Net-(D8-A1)
- T1 pad 6: Net-(D10-K) -> /PoE+ power supply/V+
- T1 pad 7: Net-(D10-K) -> /PoE+ power supply/V+
- T1 pad 9: Net-(D14-K) -> /PoE+ power supply/V-
- U10 pad 12: /ESP32-C6/T2Pb -> /ESP32-C6/SPI.SCK
- U10 pad 13: /ESP32-C6/~{RST}_{PHY} -> /ESP32-C6/~{CS}_{PHY}
- U10 pad 14: /ESP32-C6/~{CS}_{PHY} -> /ESP32-C6/T2Pb
- U10 pad 6: /ESP32-C6/SPI.SCK -> /ESP32-C6/~{RST}_{PHY}
- U10 pad 7: /ESP32-C6/SPI.MOSI -> /ESP32-C6/~{INT}_{PHY}
- U10 pad 8: /ESP32-C6/~{INT}_{PHY} -> /ESP32-C6/SPI.MOSI
- U8 pad 3: /Power supply/+12V -> +12V
- U8 pad 5: /Power supply/+12V -> +12V
- U9 pad 3: /Power supply/+12V -> +12V
- U9 pad 5: /Power supply/+12V -> +12V
Routing:
- net +12V: track 7.03 -> 124.0 mm
- net Net-(U4-~{RST}): track 4.25 -> 80.8 mm
- net Net-(U4-~{INT}): track 5.86 -> 77.5 mm
- net Net-(U4-MOSI): track 5.81 -> 76.1 mm
- net Net-(U4-MISO): track 5.77 -> 74.1 mm
- net Net-(U4-SCLK): track 5.73 -> 72.7 mm
- net GND: track 41.7 -> 108.3 mm, vias 5 -> 35
- net Net-(U4-~{SCS}): track 5.69 -> 71.3 mm
- net /PoE+ power supply/T2P: track 11.9 -> 54.3 mm
- net PGND: track 17.9 -> 58.1 mm, vias 5 -> 21
- net /PoE+ power supply/CTL: track 0.00 -> 38.8 mm
- net /PoE+ power supply/VC: track 0.00 -> 33.6 mm
- net Net-(C32-Pad1): track 0.00 -> 30.0 mm
- net Net-(R47-Pad2): track 0.00 -> 28.2 mm, vias 0 -> 2
- net /PoE+ power supply/VDD: track 33.8 -> 57.7 mm
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- added copper zone on F.Cu, net /PoE+ power supply/Q2D
- added copper zone on F.Cu, net /PoE+ power supply/Q3D
- added copper zone on F.Cu, net /PoE+ power supply/V+
- added copper zone on F.Cu, net /PoE+ power supply/V-
- added copper zone on F.Cu, net PGND

Commit message: update PCB
Parts:
- C54, C55, C57, C58, C6, L14, R22, R23, R24, R25, R26, R27, R5, R6, R8, U1: moved to B.Cu
- moved L5 81.8 mm to (98.8, 107.0), turned to -90 degrees
- moved C7 81.1 mm to (99.6, 100.2), turned to 90 degrees
- moved C8 78.3 mm to (100.7, 107.2), turned to 90 degrees
- moved C6 76.5 mm to (103.8, 108.0), turned to 180 degrees
- moved Q1 74.4 mm to (105.0, 99.3), turned to 180 degrees
- moved R6 73.6 mm to (103.1, 105.5), turned to 180 degrees
- moved R10 73.1 mm to (102.2, 99.3), turned to 90 degrees
- moved R7 73.0 mm to (103.8, 108.0)
- moved R4 71.8 mm to (107.0, 108.0), turned to 180 degrees
- moved R8 69.3 mm to (107.0, 108.0), turned to 180 degrees
- moved R11 67.5 mm to (107.9, 99.3), turned to -90 degrees
- moved R9 67.4 mm to (108.1, 104.5), turned to 90 degrees
- moved C55 59.9 mm to (107.8, 63.5), turned to 90 degrees
- moved L14 57.0 mm to (107.8, 73.0)
- moved R61 55.6 mm to (107.8, 63.5), turned to -90 degrees
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Routing:
- net /ESP32-C6/BOOT: track 0.00 -> 40.2 mm, vias 0 -> 2
- net +12V: track 124.0 -> 90.5 mm
- net GND: track 108.3 -> 141.5 mm, vias 35 -> 47
- net +3V3_ESP: track 0.00 -> 31.3 mm, vias 0 -> 1
- net +5V: track 21.1 -> 52.2 mm
- net +3.3V: track 26.2 -> 55.9 mm, vias 0 -> 1
- net /ESP32-C6/I^{2}C_{TOP}.SDA: track 0.00 -> 27.2 mm, vias 0 -> 2
- net /ESP32-C6/I^{2}C_{TOP}.SCL: track 0.00 -> 27.1 mm, vias 0 -> 2
- net /ESP32-C6/T2Pb: track 0.00 -> 24.4 mm, vias 0 -> 2
- net /Interface USB->UART/VBUS: track 0.00 -> 19.4 mm, vias 0 -> 2
- net Net-(Q1A-E1): track 0.00 -> 9.51 mm, vias 0 -> 2
- net /ESP32-C6/EN: track 0.00 -> 8.91 mm, vias 0 -> 2
- net Net-(J3-D--PadA7): track 0.00 -> 8.28 mm, vias 0 -> 1
- net Net-(U2-VBUS): track 0.00 -> 8.02 mm, vias 0 -> 1
- net +3V3_UART: track 0.00 -> 7.91 mm
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
Commit message: update
Parts:
- C56, R62: moved to B.Cu
- moved Q8 135.4 mm to (9.20, 76.1)
- moved D16 135.4 mm to (9.70, 71.9)
- moved K1 135.4 mm to (2.25, 76.0)
- moved R69 135.4 mm to (8.78, 79.6)
- moved J10 128.4 mm to (1.40, 62.9)
- moved J9 128.4 mm to (1.40, 55.0)
- moved J5 92.2 mm to (86.0, 115.4), turned to 180 degrees
- moved J7 76.6 mm to (99.2, 115.4), turned to 180 degrees
- moved J8 63.6 mm to (110.8, 115.4), turned to 180 degrees
- moved R65 35.9 mm to (95.9, 83.3)
- moved R66 34.7 mm to (95.9, 81.5)
- moved R68 33.9 mm to (95.9, 77.5)
- moved R67 33.9 mm to (95.9, 75.7)
- moved R62 29.6 mm to (98.5, 67.2)
- moved C56 27.2 mm to (98.5, 69.1), turned to 180 degrees
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Routing:
- net +3V3_ESP: track 31.3 -> 85.1 mm, vias 1 -> 2
- net /ESP32-C6/EN: track 8.91 -> 55.2 mm
- net +12V: track 90.5 -> 115.0 mm
- net /ESP32-C6/UART0.Tx: track 4.53 -> 17.3 mm
- net /ESP32-C6/UART0.Rx: track 4.59 -> 16.5 mm
- net /ESP32-C6/I^{2}C_{BOTTOM}.SCL: track 0.00 -> 11.9 mm
- net /ESP32-C6/BOOT: track 40.2 -> 50.3 mm
- net /ESP32-C6/I^{2}C_{BOTTOM}.SDA: track 0.00 -> 9.89 mm
- net /ESP32-C6/I^{2}C_{TOP}.SCL: track 27.1 -> 31.1 mm
- net /ESP32-C6/T2Pb: track 24.4 -> 27.9 mm
- net /ESP32-C6/I^{2}C_{TOP}.SDA: track 27.2 -> 28.8 mm
