File: hardware/KiCAD/mpair.kicad_pcb (KiCad board)
At the start: 2 copper layers, 100 x 102 mm, 194 parts, among them J1 PJ-063AH, J2 PJ-063AH, J3 DX07S016JA1R1500, J4 ARJP11A-MASA-B-A-EMU2, K1 G6K-2G-TR DC5, Q1 BC846B, Q2 FDMC2523P, Q3 FDS86242, Q4 CSD19534Q, Q5 FCX493, Q6 FCX493, Q7 CSD19534Q, Q8 MMBT3904, T1 PA4065NL, U1 USBLC6-2SC6, U10 ESP32-C6-WROOM-1U, U11 74AHCT1G125, U2 CP2102N, U3 ESDS314, U4 W5500, U5 TPS23754, U6 HMHA2801A, U7 PC357N, U8 TPS563208, U9 TPS563208, Y1 ECS-2520MV-250

Commit message: update
Parts:
- removed REF**: SPS30, MarPi82:SPS30
- moved J10 127.3 mm to (116.3, 117.7), turned to 90 degrees
- moved J9 116.9 mm to (100.1, 117.7), turned to 90 degrees
- moved R69 113.3 mm to (118.2, 108.9), turned to -90 degrees
- moved K1 112.5 mm to (108.2, 113.9)
- moved Q8 110.5 mm to (114.8, 108.8), turned to 180 degrees
- moved D16 105.2 mm to (108.8, 107.1)
- moved J7 79.4 mm to (70.0, 41.5), turned to 90 degrees
- moved R70 50.6 mm to (81.7, 64.1), turned to -90 degrees
- moved U11 46.6 mm to (85.4, 64.0), turned to -90 degrees
- moved J11 44.1 mm to (86.1, 69.2), turned to 180 degrees
- moved J8 26.9 mm to (84.0, 113.9), turned to 90 degrees
- moved J5 6.93 mm to (92.3, 112.4), turned to 90 degrees
Connections:
- U3 pad 1: /Interface PHY/RD+ -> /Interface PHY/RD-
- U3 pad 3: /Interface PHY/RD- -> /Interface PHY/RD+
- U3 pad 4: /Interface PHY/TD- -> /Interface PHY/TD+
- U3 pad 5: /Interface PHY/TD+ -> /Interface PHY/TD-
Routing:
- net +3.3V: track 55.9 -> 158.9 mm, vias 1 -> 4
- net GND: track 141.5 -> 208.0 mm, vias 47 -> 55
- net /ESP32-C6/I^{2}C_{CENTER}.SDA: track 6.65 -> 73.0 mm, vias 0 -> 2
- net /ESP32-C6/I^{2}C_{CENTER}.SCL: track 6.91 -> 72.8 mm, vias 0 -> 2
- net +5V: track 52.2 -> 93.3 mm, vias 0 -> 2
- net /ESP32-C6/I^{2}C_{BOTTOM}.SDA: track 9.89 -> 48.0 mm, vias 0 -> 2
- net /ESP32-C6/I^{2}C_{BOTTOM}.SCL: track 11.9 -> 49.6 mm
- net /ESP32-C6/I^{2}C_{TOP}.SCL: track 31.1 -> 68.6 mm, vias 2 -> 3
- net /ESP32-C6/I^{2}C_{TOP}.SDA: track 28.8 -> 66.2 mm, vias 2 -> 5
- net /ESP32-C6/WS2812B: track 0.00 -> 34.5 mm, vias 0 -> 4
- net /ESP32-C6/ALARM: track 0.00 -> 31.7 mm
- net /ESP32-C6/HEATER: track 0.00 -> 30.9 mm, vias 0 -> 2
- net +12V: track 115.0 -> 135.9 mm, vias 0 -> 2
- net SHIELD: track 59.2 -> 72.2 mm
- net /PoE+ power supply/VSS: track 0.14 -> 12.5 mm
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
Commit message: update
Parts:
- added H1: MountingHole, MountingHole:MountingHole_2.7mm_M2.5, F.Cu at (115.8, 22.2)
- added H2: MountingHole, MountingHole:MountingHole_2.7mm_M2.5, F.Cu at (84.3, 105.2)
- added H3: MountingHole, MountingHole:MountingHole_2.7mm_M2.5, F.Cu at (27.3, 58.1)
- added H4: MountingHole, MountingHole:MountingHole_2.7mm_M2.5, F.Cu at (27.3, 100.1)
- added REF**: SPS30, MarPi82:SPS30, F.Cu at (97.3, 39.4)
- J1, J2: footprint Connector_BarrelJack:BarrelJack_CUI_PJ-063AH_Horizontal_CircularHoles -> Connector_BarrelJack:BarrelJack_CUI_PJ-063AH_Horizontal
