File: hardware/KiCAD/PoE+_power.kicad_sch (KiCad schematic)
At the start: 68 parts, among them Q2 FDMC2523P, Q3 FDS86242, Q4 CSD19534Q, Q5 FCX493, Q6 FCX493, Q7 CSD19534Q, T1 PA4065NL, U5 TPS23754PWPR, U6 HMHA2801A, U7 PC357N4J000F

Commit message: update
Parts:
- added D6: SMBJ58CA, Diode_SMD:D_SMB, symbol Device:D_Zener_Small
- R32, R36, R41: value 100kΩ/0603 -> 100kΩ; DigiKey_Part_Number (none) -> 541-100KHCT-ND; Manufacturer_Name (none) -> CRCW0603100KFKEA; Manufacturer_Part_Number (none) -> Vishay Dale; PACKAGE (none) -> 0603; Part name RCS06031K00FKEA -> (none); Power (none) -> 0.125W, 1/8W; Tolerance (none) -> 1%
- R33: value 4,64kΩ/0603 -> 4,64kΩ; DigiKey_Part_Number (none) -> 541-4.64KHCT-ND; Manufacturer_Name (none) -> CRCW06034K64FKEA; Manufacturer_Part_Number (none) -> Vishay Dale; PACKAGE (none) -> 0603; Part name RCS06034K64FKEA -> (none); Power (none) -> 0.125W, 1/8W; Tolerance (none) -> 1%
- R34: value 69,8kΩ/0603 -> 69,8kΩ; DigiKey_Part_Number (none) -> 541-69.8KHCT-ND; Manufacturer_Name (none) -> CRCW060369K8FKEA; Manufacturer_Part_Number (none) -> Vishay Dale; PACKAGE (none) -> 0603; Part name RCS060369K8FKEA -> (none); Power (none) -> 0.125W, 1/8W; Tolerance (none) -> 1%
- R35: value 40,2kΩ/0603 -> 40,2kΩ; DigiKey_Part_Number (none) -> 541-40.2KHCT-ND; Manufacturer_Name (none) -> CRCW060340K2FKEA; Manufacturer_Part_Number (none) -> Vishay Dale; PACKAGE (none) -> 0603; Part name RCS060340K2FKEA -> (none); Power (none) -> 0.125W, 1/8W; Tolerance (none) -> 1%
- R37: value 63,4kΩ/0603 -> 63,4kΩ; DigiKey_Part_Number (none) -> 541-63.4KHCT-ND; Manufacturer_Name (none) -> CRCW060363K4FKEA; Manufacturer_Part_Number (none) -> Vishay Dale; PACKAGE (none) -> 0603; Part name RCS060363K4FKEA -> (none); Power (none) -> 0.125W, 1/8W; Tolerance (none) -> 1%
- R38, R47: value 24,9kΩ/0603 -> 24,9kΩ; DigiKey_Part_Number (none) -> 541-24.9KHCT-ND; Manufacturer_Name (none) -> CRCW060324K9FKEA; Manufacturer_Part_Number (none) -> Vishay Dale; PACKAGE (none) -> 0603; Part name RCS060324K9FKEA -> (none); Power (none) -> 0.125W, 1/8W; Tolerance (none) -> 1%
- R39, R43: value 4,7Ω/0603 -> 4,7Ω; DigiKey_Part_Number (none) -> 541-4.70HHCT-ND; Manufacturer_Name (none) -> CRCW06034R70FKEA; Manufacturer_Part_Number (none) -> Vishay Dale; PACKAGE (none) -> 0603; Part name RCS06034R70FKEA -> (none); Power (none) -> 0.125W, 1/8W; Tolerance (none) -> 1%
- R42: value 499Ω/0603 -> 499Ω; DigiKey_Part_Number (none) -> 541-499HCT-ND; Manufacturer_Name (none) -> CRCW0603499RFKEA; Manufacturer_Part_Number (none) -> Vishay Dale; PACKAGE (none) -> 0603; Part name RCS0603499RFKEA -> (none); Power (none) -> 0.125W, 1/8W; Tolerance (none) -> 1%
- R44: value 2,49kΩ/0603 -> 2,49kΩ; DigiKey_Part_Number (none) -> 541-2.49KHCT-ND; Manufacturer_Name (none) -> CRCW06032K49FKEA; Manufacturer_Part_Number (none) -> Vishay Dale; PACKAGE (none) -> 0603; Part name RCS06032K49FKEA -> (none); Power (none) -> 0.125W, 1/8W; Tolerance (none) -> 1%
- R45: DigiKey_Part_Number (none) -> 541-2740-1-ND; Manufacturer_Name (none) -> RCWE1206R100FKEA; Manufacturer_Part_Number (none) -> Vishay Dale; PACKAGE (none) -> 1206; Part name RCWE1206R100FKEA -> (none); Power (none) -> 0.5W, 1/2W; Tolerance (none) -> 1%
- R46, R48: value 2kΩ/0603 -> 2kΩ; DigiKey_Part_Number (none) -> 541-2.00KHCT-ND; Manufacturer_Name (none) -> CRCW06032K00FKEA; Manufacturer_Part_Number (none) -> Vishay Dale; PACKAGE (none) -> 0603; Part name RCS06032K00FKEA -> (none); Tolerance (none) -> 1%
- R50: footprint Resistor_SMD:R_0603_1608Metric -> Resistor_SMD:R_0805_2012Metric; DigiKey_Part_Number (none) -> 541-2.00KCCT-ND; Manufacturer_Name (none) -> CRCW08052K00FKEA; Manufacturer_Part_Number (none) -> Vishay Dale; PACKAGE (none) -> 0805; Part name RCS06032K00FKEA -> (none); Power 0.25W, 1/4 -> 0.25W, 1/4W; Tolerance (none) -> 1%
- R51: renamed from R54; footprint Resistor_SMD:R_0603_1608Metric -> Resistor_SMD:R_0805_2012Metric; DigiKey_Part_Number (none) -> 541-2.00KCCT-ND; Manufacturer_Name (none) -> CRCW08052K00FKEA; Manufacturer_Part_Number (none) -> Vishay Dale; PACKAGE (none) -> 0805; Part name RCS06032K00FKEA -> (none); Power 0.25W, 1/4 -> 0.25W, 1/4W; Tolerance (none) -> 1%
- R54: renamed from R53; value 2,61kΩ/0603 -> 2,61kΩ; DigiKey_Part_Number (none) -> 541-2.61KHCT-ND; Manufacturer_Name (none) -> CRCW06032K61FKEA; Manufacturer_Part_Number (none) -> Vishay Dale; PACKAGE (none) -> 0805; Part name RCS06032K61FKEA -> (none); Power (none) -> 0.25W, 1/4W; Tolerance (none) -> 1%
- T1: DigiKey_Part_Number (none) -> PA4065NL-ND; Part name PA4065NL -> (none)
- U5: value TPS23754PWPR -> TPS23754; DigiKey_Part_Number (none) -> 296-39367-1-ND; Manufacturer_Name (none) -> TPS23754PWPR; Manufacturer_Part_Number (none) -> Texas Instruments; PACKAGE TSSOP-20 -> 20-PowerTSSOP; Part name TPS23754PWPR -> (none)
- U6: DigiKey_Part_Number (none) -> HMHA2801AR2VCT-ND; Manufacturer_Name (none) -> HMHA2801AR2V; Manufacturer_Part_Number (none) -> onsemi; PACKAGE (none) -> 4-SOIC (0.173", 4.40mm Width); Part name HMHA2801A -> (none)
- U7: value PC357N4J000F -> PC357N; DigiKey_Part_Number (none) -> 1855-1022-1-ND; Manufacturer_Name (none) -> PC357N4J000F; Manufacturer_Part_Number (none) -> SHARP/Socle Technology; PACKAGE (none) -> 4-SMD, Gull Wing; Part name PC357N4J000F -> (none)
- renumbered C39 to C38, C38 to C39, D9 to D10, D10 to D11, D11 to D12, D12 to D13, D13 to D14, D14 to D15, D6 to D7, D7 to D8, D8 to D9, R51 to R52, R52 to R53
Connections:
- net PGND: now also D6.1 (K)
- net VSS: now reaches C24.2, D5.2 (A), L8.3, R37.2, U5.10 (VSS), U5.21 (EPAD)
- net VSS: now also D6.2 (A)
- net VDD: now reaches C24.1, C27.1, D5.1 (K), L8.2, L9.1, R38.1, U5.11 (VDD1), U5.12 (VDD)
- net POE- renamed AUXGND

Commit message: update
Parts:
- U7: footprint Package_SO:SOIC-4_4.55x3.7mm_P2.54mm -> Package_SO:OnSemi_751EP_SOIC-4_3.9x4.725mm_P2.54mm
Changed lines of the file:
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@@
 			)
 		)
-		(property "Footprint" "Package_SO:SOIC-4_4.55x3.7mm_P2.54mm"
+		(property "Footprint" "Package_SO:OnSemi_751EP_SOIC-4_3.9x4.725mm_P2.54mm"
 			(at 157.48 129.54 0)
 			(effects

Commit message: update
Parts:
- removed D10, D14, D7, D8, D9: MMBD4148, Package_TO_SOT_SMD:SC-59, symbol Device:D_Small
- added D10, D14, D7: MMBD4148, Package_TO_SOT_SMD:SC-59, symbol MarPi82:MMBD4148
- added D8: MMBD4148CC, Package_TO_SOT_SMD:SC-59, symbol MarPi82:MMBD4148CC
Connections:
- net PGND: now also D7.3 (K)
- net Q2D: now reaches C26.2, Q2.D
- net at C25.1, Q2.G, R40.2: now also D7.1 (A)
- net VB: now reaches C29.2, C30.1, R41.1, R46.2, U5.2 (VB)
- net CTL: now reaches R42.1, R46.1, U5.1 (CTL), U6.4
- net T2P: now reaches U5.20 (T2P), U7.2
- net VC: now reaches C28.1, C31.1, L10.1, R47.1, U5.6 (VC)
- net GATE2: now reaches R39.2, U5.7 (GAT2)
- net Q3D: now reaches C26.1, Q3.D, T1.2
- net V-: now reaches C38.1, Q4.D, Q6.2 (C), R51.1, T1.10, T1.9
- net V-: now also D14.3 (K)
- net at Q4.G, Q5.3 (E): now also D10.1 (A)
- net at L10.2: now also D8.3 (K)
- net at T1.4: now also D8.1 (A1)
- net V+: now reaches L11.1, Q5.2 (C), Q7.D, R50.1, T1.6, T1.7
- net V+: now also D10.3 (K)
- net at Q6.3 (E), Q7.G: now also D14.1 (A)
- net at C28.2: now also D8.2 (A2)

Commit message: update
Other:
- title: Czujnik parametrów środowiskowych -> Enviromental parameters multi-sensor
Changed lines of the file:
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@@
 	(paper "A4")
 	(title_block
-		(title "Czujnik parametrów środowiskowych")
+		(title "Enviromental parameters multi-sensor")
 		(date "2026-01-20")
 		(rev "1.0")
