File: hardware/KiCAD/esp32-c6.kicad_sch (KiCad schematic)
At the start: 18 parts, among them SW1 EN, SW2 BOOT, U10 ESP32-C6-WROOM-1U-N16

Commit message: update
Parts:
- R63, R64, R65, R66, R67, R68: value 4,7kΩ/0603 -> 4,7kΩ; DigiKey_Part_Number (none) -> 541-4.70KHCT-ND; Manufacturer_Name (none) -> CRCW06034K70FKEA; Manufacturer_Part_Number (none) -> Vishay Dale; PACKAGE (none) -> 0805; Part name RCS06034K70FKEA -> (none); Power (none) -> 0.25W, 1/4W; Tolerance (none) -> 1%
- SW1: value EN -> ~; DigiKey_Part_Number (none) -> 450-1140-ND; Label (none) -> EN; Manufacturer_Name (none) -> FSMSM; Manufacturer_Part_Number (none) -> TE Connectivity; Part name FSMSM -> (none)
- SW2: value BOOT -> ~; DigiKey_Part_Number (none) -> 450-1140-ND; Label (none) -> BOOT; Manufacturer_Name (none) -> FSMSM; Manufacturer_Part_Number (none) -> TE Connectivity; Part name FSMSM -> (none)
- U10: value ESP32-C6-WROOM-1U-N16 -> ESP32-C6-WROOM-1U; DigiKey_Part_Number (none) -> 1965-ESP32-C6-WROOM-1U-N8CT-ND; Manufacturer_Name (none) -> ESP32-C6-WROOM-1U-N8; Manufacturer_Part_Number (none) -> Espressif Systems; PACKAGE (none) -> 37-SMD Module; Part name ESP32-C6-WROOM-1U-N16 -> (none)

Commit message: update
Changed lines of the file:
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@@
 					(size 0.762 0.762)
 				)
+				(hide yes)
 			)
 		)
@@
 					(size 1.524 1.524)
 				)
+				(hide yes)
 			)
 		)
@@
 					(size 0.762 0.762)
 				)
+				(hide yes)
 			)
 		)
@@
 				)
 				(justify left)
+				(hide yes)
 			)
 		)
@@
 					(size 0.762 0.762)
 				)
+				(hide yes)
 			)
 		)
@@
 					(size 0.762 0.762)
 				)
+				(hide yes)
 			)
 		)
@@
 				)
 				(justify left)
+				(hide yes)
 			)
 		)
@@
 					(size 0.762 0.762)
 				)
+				(hide yes)
 			)
 		)
@@
 				)
 				(justify left)
+				(hide yes)
 			)
 		)
@@
 					(size 0.762 0.762)
 				)
+				(hide yes)
 			)
 		)
@@
 					(size 0.762 0.762)
 				)
+				(hide yes)
 			)
 		)
@@
 					(size 0.762 0.762)
 				)
+				(hide yes)
 			)
 		)
@@
 					(size 0.762 0.762)
 				)
+				(hide yes)
 			)
 		)
@@
 				)
 				(justify left)
+				(hide yes)
 			)
 		)
@@
 				)
 				(justify left)
+				(hide yes)
 			)
 		)
@@
 				)
 				(justify left)
+				(hide yes)
 			)
 		)
@@
 					(size 0.762 0.762)
 				)
+				(hide yes)
 			)
 		)
@@
 					(size 0.762 0.762)
 				)
+				(hide yes)
 			)
 		)
@@
 					(size 0.762 0.762)
 				)
+				(hide yes)
 			)
 		)
@@
 				)
 				(justify left)
+				(hide yes)
 			)
 		)
@@
 				)
 				(justify left)
+				(hide yes)
 			)
 		)
@@
 				)
 				(justify left)
+				(hide yes)
 			)
 		)
@@
 				)
 				(justify left)
+				(hide yes)
 			)
 		)
@@
 				)
 				(justify left)
+				(hide yes)
 			)
 		)
@@
 					(size 0.762 0.762)
 				)
+				(hide yes)
 			)
 		)
@@
 					(size 0.762 0.762)
 				)
+				(hide yes)
 			)
 		)
@@
 				)
 				(justify left)
+				(hide yes)
 			)
 		)
@@
 				)
 				(justify left)
+				(hide yes)
 			)
 		)
@@
 					(size 0.762 0.762)
 				)
+				(hide yes)
 			)
 		)
@@
 				)
 				(justify left)
+				(hide yes)
 			)
 		)
@@
 				)
 				(justify left)
+				(hide yes)
 			)
 		)

Commit message: update
Changed lines of the file:
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@@
 					(size 0.762 0.762)
 				)
-				(hide yes)
 			)
 		)
@@
 					(size 1.524 1.524)
 				)
-				(hide yes)
 			)
 		)
@@
 					(size 1.27 1.27)
 				)
-				(hide yes)
 			)
 		)
@@
 					(size 0.762 0.762)
 				)
-				(hide yes)
 			)
 		)
@@
 				)
 				(justify left)
-				(hide yes)
 			)
 		)
@@
 					(size 0.762 0.762)
 				)
-				(hide yes)
 			)
 		)
@@
 					(size 0.762 0.762)
 				)
-				(hide yes)
 			)
 		)
@@
 				)
 				(justify left)
-				(hide yes)
 			)
 		)
@@
 					(size 0.762 0.762)
 				)
-				(hide yes)
 			)
 		)
@@
 				)
 				(justify left)
-				(hide yes)
 			)
 		)
@@
 					(size 0.762 0.762)
 				)
-				(hide yes)
 			)
 		)
@@
 					(size 0.762 0.762)
 				)
-				(hide yes)
 			)
 		)
@@
 					(size 0.762 0.762)
 				)
-				(hide yes)
 			)
 		)
@@
 					(size 0.762 0.762)
 				)
-				(hide yes)
 			)
 		)
@@
 					(size 1.27 1.27)
 				)
-				(hide yes)
 			)
 		)
@@
 				)
 				(justify left)
-				(hide yes)
 			)
 		)
@@
 				)
 				(justify left)
-				(hide yes)
 			)
 		)
@@
 				)
 				(justify left)
-				(hide yes)
 			)
 		)
@@
 					(size 0.762 0.762)
 				)
-				(hide yes)
 			)
 		)
@@
 					(size 0.762 0.762)
 				)
-				(hide yes)
 			)
 		)
@@
 					(size 0.762 0.762)
 				)
-				(hide yes)
 			)
 		)
@@
 				)
 				(justify left)
-				(hide yes)
 			)
 		)
@@
 				)
 				(justify left)
-				(hide yes)
 			)
 		)
@@
 				)
 				(justify left)
-				(hide yes)
 			)
 		)
@@
 				)
 				(justify left)
-				(hide yes)
 			)
 		)
@@
 				)
 				(justify left)
-				(hide yes)
 			)
 		)
@@
 					(size 0.762 0.762)
 				)
-				(hide yes)
 			)
 		)
@@
 					(size 0.762 0.762)
 				)
-				(hide yes)
 			)
 		)
@@
 				)
 				(justify left)
-				(hide yes)
 			)
 		)
@@
 				)
 				(justify left)
-				(hide yes)
 			)
 		)
@@
 					(size 0.762 0.762)
 				)
-				(hide yes)
 			)
 		)
@@
 				)
 				(justify left)
-				(hide yes)
 			)
 		)
@@
 				)
 				(justify left)
-				(hide yes)
 			)
 		)

Commit message: update
Connections:
- net SPI.MOSI: now also U10.8 (IO40); no longer U10.7 (IO7)
- net SPI.SCK: now also U10.12 (IO11); no longer U10.6 (IO6)
- net T2Pb: now also U10.14 (IO13); no longer U10.12 (IO11)
- net ~{CS}_{PHY}: now also U10.13 (IO12); no longer U10.14 (IO13)
- net ~{INT}_{PHY}: now also U10.7 (IO7); no longer U10.8 (IO40)
- net ~{RST}_{PHY}: now also U10.6 (IO6); no longer U10.13 (IO12)
Other:
- moved on the sheet: C56, R62

Commit message: update
Other:
- title: Czujnik parametrów środowiskowych -> Enviromental parameters multi-sensor
Changed lines of the file:
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@@
 	(paper "A4")
 	(title_block
-		(title "Czujnik parametrów środowiskowych")
+		(title "Enviromental parameters multi-sensor")
 		(date "2026-01-20")
 		(rev "1.0")
