File: hardware/KiCAD/mini_relay.kicad_sch (KiCad schematic)
At the start: 4 parts, among them K1 G6K-2G-TR DC5, Q8 MMBT3904

Commit message: update
Parts:
- R69: value 4,7kΩ/0603 -> 4,7kΩ; DigiKey_Part_Number (none) -> 541-4.70KHCT-ND; Manufacturer_Name (none) -> CRCW06034K70FKEA; Manufacturer_Part_Number (none) -> Vishay Dale; PACKAGE (none) -> 0805; Part name RCS06034K70FKEA -> (none); Power (none) -> 0.25W, 1/4W; Tolerance (none) -> 1%
- renumbered D15 to D16
Changed lines of the file:
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@@
-			)
-		)
-		(property "Part name" ""
-			(at 152.4 86.36 0)
-			(effects
-				(font
-					(size 0.762 0.762)
-				)
-				(hide yes)
 			)
 		)
@@
 		)
 		(property "Tolerance" ""
+			(at 152.4 86.36 0)
+			(effects
+				(font
+					(size 1.27 1.27)
+				)
+				(hide yes)
+			)
+		)
+		(property "MPN" ""
+			(at 152.4 86.36 0)
+			(effects
+				(font
+					(size 1.27 1.27)
+				)
+				(hide yes)
+			)
+		)
+		(property "OC_FARNELL" ""
+			(at 152.4 86.36 0)
+			(effects
+				(font
+					(size 1.27 1.27)
+				)
+				(hide yes)
+			)
+		)
+		(property "OC_NEWARK" ""
+			(at 152.4 86.36 0)
+			(effects
+				(font
+					(size 1.27 1.27)
+				)
+				(hide yes)
+			)
+		)
+		(property "SUPPLIER" ""
 			(at 152.4 86.36 0)
 			(effects
@@
 		(dnp no)
 		(fields_autoplaced yes)
-		(property "Reference" "D15"
+		(property "Reference" "D16"
 			(at 127 86.3599 90)
 			(effects
@@
 			)
 		)
-		(property "Part name" ""
-			(at 124.46 87.63 90)
-			(effects
-				(font
-					(size 0.762 0.762)
-				)
-				(hide yes)
-			)
-		)
 		(property "DigiKey_Part_Number" "31-1N4148W-7-F-WCT-ND"
 			(at 124.46 87.63 90)
@@
 		)
 		(property "Tolerance" ""
+			(at 124.46 87.63 90)
+			(effects
+				(font
+					(size 1.27 1.27)
+				)
+				(hide yes)
+			)
+		)
+		(property "MPN" ""
+			(at 124.46 87.63 90)
+			(effects
+				(font
+					(size 1.27 1.27)
+				)
+				(hide yes)
+			)
+		)
+		(property "OC_FARNELL" ""
+			(at 124.46 87.63 90)
+			(effects
+				(font
+					(size 1.27 1.27)
+				)
+				(hide yes)
+			)
+		)
+		(property "OC_NEWARK" ""
+			(at 124.46 87.63 90)
+			(effects
+				(font
+					(size 1.27 1.27)
+				)
+				(hide yes)
+			)
+		)
+		(property "SUPPLIER" ""
 			(at 124.46 87.63 90)
 			(effects
@@
 			(project ""
 				(path "/c7dbdcbe-6da7-4d67-a2bd-18f9bca31cdc/5c895c17-692e-46ff-ba12-a526f1167785"
-					(reference "D15")
+					(reference "D16")
 					(unit 1)
 				)
@@
 			)
 		)
-		(property "Value" "4,7kΩ/0603"
+		(property "Value" "4,7kΩ"
 			(at 135.382 103.632 90)
 			(effects
@@
 			)
 		)
-		(property "Part name" "RCS06034K70FKEA"
-			(at 132.08 105.41 0)
-			(effects
-				(font
-					(size 0.762 0.762)
-				)
-				(hide yes)
-			)
-		)
-		(property "DigiKey_Part_Number" ""
+		(property "DigiKey_Part_Number" "541-4.70KHCT-ND"
 			(at 132.08 105.41 90)
 			(effects
@@
 			)
 		)
-		(property "Power" ""
-			(at 132.08 105.41 90)
-			(effects
-				(font
-					(size 1.27 1.27)
-				)
-				(hide yes)
-			)
-		)
-		(property "Tolerance" ""
+		(property "Power" "0.25W, 1/4W"
+			(at 132.08 105.41 90)
+			(effects
+				(font
+					(size 1.27 1.27)
+				)
+				(hide yes)
+			)
+		)
+		(property "Tolerance" "1%"
+			(at 132.08 105.41 90)
+			(effects
+				(font
+					(size 1.27 1.27)
+				)
+				(hide yes)
+			)
+		)
+		(property "Manufacturer_Name" "CRCW06034K70FKEA"
+			(at 132.08 105.41 90)
+			(effects
+				(font
+					(size 1.27 1.27)
+				)
+				(hide yes)
+			)
+		)
+		(property "Manufacturer_Part_Number" "Vishay Dale"
+			(at 132.08 105.41 90)
+			(effects
+				(font
+					(size 1.27 1.27)
+				)
+				(hide yes)
+			)
+		)
+		(property "PACKAGE" "0805"
+			(at 132.08 105.41 90)
+			(effects
+				(font
+					(size 1.27 1.27)
+				)
+				(hide yes)
+			)
+		)
+		(property "MPN" ""
+			(at 132.08 105.41 90)
+			(effects
+				(font
+					(size 1.27 1.27)
+				)
+				(hide yes)
+			)
+		)
+		(property "OC_FARNELL" ""
+			(at 132.08 105.41 90)
+			(effects
+				(font
+					(size 1.27 1.27)
+				)
+				(hide yes)
+			)
+		)
+		(property "OC_NEWARK" ""
+			(at 132.08 105.41 90)
+			(effects
+				(font
+					(size 1.27 1.27)
+				)
+				(hide yes)
+			)
+		)
+		(property "SUPPLIER" ""
 			(at 132.08 105.41 90)
 			(effects
@@
 			)
 		)
-		(property "Part name" ""
-			(at 139.7 105.41 0)
-			(effects
-				(font
-					(size 0.762 0.762)
-				)
-				(hide yes)
-			)
-		)
 		(property "DigiKey_Part_Number" "1801-MMBT3904HRFGCT-ND"
 			(at 139.7 105.41 0)
@@
 		)
 		(property "Tolerance" ""
+			(at 139.7 105.41 0)
+			(effects
+				(font
+					(size 1.27 1.27)
+				)
+				(hide yes)
+			)
+		)
+		(property "MPN" ""
+			(at 139.7 105.41 0)
+			(effects
+				(font
+					(size 1.27 1.27)
+				)
+				(hide yes)
+			)
+		)
+		(property "OC_FARNELL" ""
+			(at 139.7 105.41 0)
+			(effects
+				(font
+					(size 1.27 1.27)
+				)
+				(hide yes)
+			)
+		)
+		(property "OC_NEWARK" ""
+			(at 139.7 105.41 0)
+			(effects
+				(font
+					(size 1.27 1.27)
+				)
+				(hide yes)
+			)
+		)
+		(property "SUPPLIER" ""
 			(at 139.7 105.41 0)
 			(effects
@@
 		(on_board yes)
 		(dnp no)
-		(property "Reference" "#PWR091"
+		(property "Reference" "#PWR092"
 			(at 124.46 102.87 0)
 			(effects
@@
 			(project "mpair"
 				(path "/c7dbdcbe-6da7-4d67-a2bd-18f9bca31cdc/5c895c17-692e-46ff-ba12-a526f1167785"
-					(reference "#PWR091")
+					(reference "#PWR092")
 					(unit 1)
 				)
@@
 		(on_board yes)
 		(dnp no)
-		(property "Reference" "#PWR092"
+		(property "Reference" "#PWR093"
 			(at 142.24 123.19 0)
 			(effects
@@
 			(project "mpair"
 				(path "/c7dbdcbe-6da7-4d67-a2bd-18f9bca31cdc/5c895c17-692e-46ff-ba12-a526f1167785"
-					(reference "#PWR092")
+					(reference "#PWR093")
 					(unit 1)
 				)

Commit message: update
Changed lines of the file:
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@@
 				)
 				(justify left)
+				(hide yes)
 			)
 		)
@@
 				)
 				(justify left)
+				(hide yes)
 			)
 		)
@@
 				)
 				(justify left)
+				(hide yes)
 			)
 		)
@@
 				)
 				(justify left)
+				(hide yes)
 			)
 		)
@@
 					(size 0.762 0.762)
 				)
+				(hide yes)
 			)
 		)
@@
 					(size 0.762 0.762)
 				)
-			)
-		)
+				(hide yes)
+			)
+		)

Commit message: update
Changed lines of the file:
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@@
 				)
 				(justify left)
-				(hide yes)
 			)
 		)
@@
 				)
 				(justify left)
-				(hide yes)
 			)
 		)
@@
 				)
 				(justify left)
-				(hide yes)
 			)
 		)
@@
 				)
 				(justify left)
-				(hide yes)
 			)
 		)
@@
 					(size 0.762 0.762)
 				)
-				(hide yes)
 			)
 		)
@@
 					(size 0.762 0.762)
 				)
-				(hide yes)
-			)
-		)
+			)
+		)

Commit message: update
Other:
- title: Czujnik parametrów środowiskowych -> Enviromental parameters multi-sensor
Changed lines of the file:
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@@
 	(paper "A4")
 	(title_block
-		(title "Czujnik parametrów środowiskowych")
+		(title "Enviromental parameters multi-sensor")
 		(date "2026-01-20")
 		(rev "1.0")
