File: hardware/KiCAD/phy.kicad_sch (KiCad schematic)
At the start: 43 parts, among them U3 ESDS314DBVR, U4 W5500, Y1 ECS-2520MV-250

Commit message: update
Parts:
- R18: value 12,4kΩ/0603 -> 12,4kΩ; DigiKey_Part_Number (none) -> 541-12.4KHCT-ND; Manufacturer_Name (none) -> CRCW060312K4FKEA; Manufacturer_Part_Number (none) -> Vishay Dale; PACKAGE (none) -> 0603; Part name RCS060312K4FKEA -> (none); Power (none) -> 0.125W, 1/8W; Tolerance (none) -> 1%
- R19, R20: value 330Ω/0603 -> 330Ω; DigiKey_Part_Number (none) -> 541-330HCT-ND; Manufacturer_Name (none) -> CRCW0603330RFKEA; Manufacturer_Part_Number (none) -> Vishay Dale; PACKAGE (none) -> 0603; Part name RCS0603330RFKEA -> (none); Power (none) -> 0.125W, 1/8W; Tolerance (none) -> 1%
- R24: value 33Ω/0603 -> 33Ω; DigiKey_Part_Number (none) -> 541-33.0HCT-ND; Manufacturer_Name (none) -> CRCW060333R0FKEA; Manufacturer_Part_Number (none) -> Vishay Dale; PACKAGE (none) -> 0603; Part name RCS060333R0FKEA -> (none); Power (none) -> 0.125W, 1/8W; Tolerance (none) -> 1%
- RN1: DigiKey_Part_Number (none) -> Y43R3CT-ND; Manufacturer_Name (none) -> EXB-V8V3R3JV; Manufacturer_Part_Number (none) -> Panasonic Electronic Components; PACKAGE (none) -> 1206; Part name EXB-V8V3R3JV -> (none); Power (none) -> 62.5mW; Tolerance (none) -> 5%
- U3: value ESDS314DBVR -> ESDS314; footprint MarPi82:DBV0005A_N -> Package_TO_SOT_SMD:SOT-23-5; DigiKey_Part_Number (none) -> 296-ESDS314DBVRCT-ND; Manufacturer_Name (none) -> ESDS314DBVR; Manufacturer_Part_Number (none) -> Texas Instruments; PACKAGE (none) -> SOT-23-5; Part name ESDS314DBVR -> (none)
- U4: DigiKey_Part_Number (none) -> 1278-W5500CT-ND; Manufacturer_Name (none) -> W5500; Manufacturer_Part_Number (none) -> WIZnet; PACKAGE (none) -> 48-LQFP; Part name W5500 -> (none)
- Y1: DigiKey_Part_Number (none) -> XC2752CT-ND; Manufacturer_Name (none) -> ECS-2520MV-250-CN-TR; Manufacturer_Part_Number (none) -> ECS Inc.; PACKAGE (none) -> 4-SMD, No Lead; Part name ECS-2520MV-250-BN-TR -> (none)

Commit message: update
Changed lines of the file:
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@@
 					(size 0.762 0.762)
 				)
+				(hide yes)
 			)
 		)
@@
 					(size 1.27 1.27)
 				)
+				(hide yes)
 			)
 		)
@@
 					(size 1.27 1.27)
 				)
+				(hide yes)
 			)
 		)
@@
 				)
 				(justify left)
+				(hide yes)
 			)
 		)
@@
 					(size 1.27 1.27)
 				)
+				(hide yes)
 			)
 		)
@@
 				)
 				(justify left)
+				(hide yes)
 			)
 		)
@@
 					(size 1.27 1.27)
 				)
+				(hide yes)
 			)
 		)
@@
 					(size 0.762 0.762)
 				)
+				(hide yes)
 			)
 		)
@@
 					(size 0.762 0.762)
 				)
+				(hide yes)
 			)
 		)
@@
 				)
 				(justify left)
+				(hide yes)
 			)
 		)
@@
 					(size 0.762 0.762)
 				)
+				(hide yes)
 			)
 		)
@@
 				)
 				(justify left)
+				(hide yes)
 			)
 		)
@@
 				)
 				(justify left)
+				(hide yes)
 			)
 		)
@@
 					(size 1.27 1.27)
 				)
+				(hide yes)
 			)
 		)
@@
 				)
 				(justify left)
+				(hide yes)
 			)
 		)
@@
 				)
 				(justify left)
+				(hide yes)
 			)
 		)
@@
 				)
 				(justify left)
+				(hide yes)
 			)
 		)
@@
 					(size 0.762 0.762)
 				)
+				(hide yes)
 			)
 		)
@@
 				)
 				(justify left)
+				(hide yes)
 			)
 		)
@@
 				)
 				(justify left)
+				(hide yes)
 			)
 		)
@@
 					(size 1.27 1.27)
 				)
+				(hide yes)
 			)
 		)
@@
 					(size 1.27 1.27)
 				)
+				(hide yes)
 			)
 		)
@@
 					(size 0.762 0.762)
 				)
+				(hide yes)
 			)
 		)
@@
 				)
 				(justify left)
+				(hide yes)
 			)
 		)
@@
 				)
 				(justify left)
+				(hide yes)
 			)
 		)
@@
 				)
 				(justify left)
+				(hide yes)
 			)
 		)
@@
 				)
 				(justify left)
+				(hide yes)
 			)
 		)
@@
 				)
 				(justify left)
+				(hide yes)
 			)
 		)
@@
 				)
 				(justify left)
+				(hide yes)
 			)
 		)
@@
 				)
 				(justify left)
+				(hide yes)
 			)
 		)
@@
 				)
 				(justify left)
+				(hide yes)
 			)
 		)
@@
 				)
 				(justify left)
+				(hide yes)
 			)
 		)
@@
 					(size 1.27 1.27)
 				)
+				(hide yes)
 			)
 		)
@@
 				)
 				(justify left)
+				(hide yes)
 			)
 		)
@@
 				)
 				(justify left)
+				(hide yes)
 			)
 		)
@@
 					(size 1.27 1.27)
 				)
+				(hide yes)
 			)
 		)
@@
 				)
 				(justify left)
+				(hide yes)
 			)
 		)
@@
 					(size 1.27 1.27)
 				)
+				(hide yes)
 			)
 		)
@@
 					(size 1.27 1.27)
 				)
+				(hide yes)
 			)
 		)
@@
 				)
 				(justify left)
+				(hide yes)
 			)
 		)
@@
 				)
 				(justify left)
+				(hide yes)
 			)
 		)
@@
 					(size 0.762 0.762)
 				)
+				(hide yes)
 			)
 		)
@@
 					(size 1.27 1.27)
 				)
+				(hide yes)
 			)
 		)
@@
 					(size 1.27 1.27)
 				)
+				(hide yes)
 			)
 		)
@@
 				)
 				(justify left)
+				(hide yes)
 			)
 		)
@@
 				)
 				(justify left)
+				(hide yes)
 			)
 		)
@@
 				)
 				(justify left)
+				(hide yes)
 			)
 		)
@@
 				)
 				(justify left)
+				(hide yes)
 			)
 		)
@@
 				)
 				(justify left)
+				(hide yes)
 			)
 		)
@@
 					(size 1.27 1.27)
 				)
+				(hide yes)
 			)
 		)
@@
 				)
 				(justify left)
+				(hide yes)
 			)
 		)
@@
 				)
 				(justify left)
+				(hide yes)
 			)
 		)
@@
 				)
 				(justify left)
+				(hide yes)
 			)
 		)
@@
 					(size 1.27 1.27)
 				)
+				(hide yes)
 			)
 		)
@@
 					(size 0.762 0.762)
 				)
+				(hide yes)
 			)
 		)
@@
 					(size 1.27 1.27)
 				)
+				(hide yes)
 			)
 		)
@@
 				)
 				(justify left)
+				(hide yes)
 			)
 		)
@@
 				)
 				(justify left)
+				(hide yes)
 			)
 		)
@@
 				)
 				(justify left)
+				(hide yes)
 			)
 		)
@@
 				)
 				(justify left)
+				(hide yes)
 			)
 		)
@@
 					(size 0.762 0.762)
 				)
+				(hide yes)
 			)
 		)
@@
 				)
 				(justify left)
+				(hide yes)
 			)
 		)
@@
 				)
 				(justify left)
+				(hide yes)
 			)
 		)
@@
 				)
 				(justify left)
+				(hide yes)
 			)
 		)

Commit message: update
Connections:
- net RD+: now also C12.1; no longer C11.1
- net RD-: now also C11.1; no longer C12.1
- net TD+: now also R14.2, RN1.2 (R2.1), U3.5 (I_O4); no longer R16.2, RN1.1 (R1.1), U3.4 (I_O3)
- net TD-: now also R16.2, RN1.1 (R1.1), U3.4 (I_O3); no longer R14.2, RN1.2 (R2.1), U3.5 (I_O4)
- net at D4.1 (A1), RN1.5 (R4.2): now also U4.6 (RXP); no longer U4.5 (RXN)
- net at D4.2 (A2), RN1.6 (R3.2): now also U4.5 (RXN); no longer U4.6 (RXP)
- net at D3.2 (A2), RN1.7 (R2.2): now also U4.2 (TXP); no longer U4.1 (TXN)
- net at D3.1 (A1), RN1.8 (R1.2): now also U4.1 (TXN); no longer U4.2 (TXP)

Commit message: update
Connections:
- net RD+: now also U3.3 (I_O2); no longer U3.1 (I_O1)
- net RD-: now also U3.1 (I_O1); no longer U3.3 (I_O2)
- net TD+: now also U3.4 (I_O3); no longer U3.5 (I_O4)
- net TD-: now also U3.5 (I_O4); no longer U3.4 (I_O3)
Changed lines of the file:
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@@
+	(wire
+		(pts
+			(xy 86.36 69.85) (xy 99.06 69.85)
+		)
+		(stroke
+			(width 0)
+			(type default)
+		)
+	)
 	(wire
 		(pts
@@
 	(wire
 		(pts
+			(xy 91.44 40.64) (xy 91.44 43.18)
+		)
+		(stroke
+			(width 0)
+			(type default)
+		)
+	)
+	(wire
+		(pts
 			(xy 190.5 104.14) (xy 190.5 105.41)
 		)
@@
 	(wire
 		(pts
-			(xy 91.44 67.31) (xy 91.44 69.85)
-		)
-		(stroke
-			(width 0)
-			(type default)
-		)
-	)
-	(wire
-		(pts
 			(xy 142.24 86.36) (xy 144.78 86.36)
 		)
@@
 	(wire
 		(pts
+			(xy 86.36 41.91) (xy 86.36 43.18)
+		)
+		(stroke
+			(width 0)
+			(type default)
+		)
+	)
+	(wire
+		(pts
 			(xy 120.65 69.85) (xy 120.65 67.31)
 		)
@@
 	(wire
 		(pts
-			(xy 86.36 41.91) (xy 101.6 41.91)
-		)
-		(stroke
-			(width 0)
-			(type default)
-		)
-	)
-	(wire
-		(pts
 			(xy 129.54 57.15) (xy 135.89 57.15)
 		)
@@
 	(wire
 		(pts
+			(xy 91.44 40.64) (xy 101.6 40.64)
+		)
+		(stroke
+			(width 0)
+			(type default)
+		)
+	)
+	(wire
+		(pts
 			(xy 165.1 137.16) (xy 162.56 137.16)
 		)
@@
 	(wire
 		(pts
+			(xy 100.33 41.91) (xy 86.36 41.91)
+		)
+		(stroke
+			(width 0)
+			(type default)
+		)
+	)
+	(wire
+		(pts
 			(xy 120.65 77.47) (xy 120.65 80.01)
 		)
@@
 	(wire
 		(pts
-			(xy 101.6 41.91) (xy 101.6 85.09)
+			(xy 86.36 69.85) (xy 86.36 67.31)
+		)
+		(stroke
+			(width 0)
+			(type default)
+		)
+	)
+	(wire
+		(pts
+			(xy 101.6 40.64) (xy 101.6 85.09)
 		)
 		(stroke
@@
 	(wire
 		(pts
+			(xy 91.44 71.12) (xy 91.44 67.31)
+		)
+		(stroke
+			(width 0)
+			(type default)
+		)
+	)
+	(wire
+		(pts
 			(xy 120.65 100.33) (xy 115.57 100.33)
 		)
@@
 	(wire
 		(pts
-			(xy 100.33 43.18) (xy 100.33 90.17)
+			(xy 100.33 41.91) (xy 100.33 90.17)
 		)
 		(stroke
@@
 	(wire
 		(pts
-			(xy 91.44 43.18) (xy 100.33 43.18)
-		)
-		(stroke
-			(width 0)
-			(type default)
-		)
-	)
-	(wire
-		(pts
 			(xy 190.5 99.06) (xy 190.5 101.6)
 		)
@@
 	(wire
 		(pts
-			(xy 86.36 43.18) (xy 86.36 41.91)
-		)
-		(stroke
-			(width 0)
-			(type default)
-		)
-	)
-	(wire
-		(pts
 			(xy 205.74 105.41) (xy 205.74 101.6)
 		)
@@
 	(wire
 		(pts
-			(xy 86.36 67.31) (xy 86.36 71.12)
-		)
-		(stroke
-			(width 0)
-			(type default)
-		)
-	)
-	(wire
-		(pts
 			(xy 142.24 81.28) (xy 142.24 82.55)
 		)
@@
 	(wire
 		(pts
-			(xy 86.36 71.12) (xy 97.79 71.12)
-		)
-		(stroke
-			(width 0)
-			(type default)
-		)
-	)
-	(wire
-		(pts
 			(xy 176.53 114.3) (xy 176.53 116.84)
 		)
@@
 	(wire
 		(pts
-			(xy 91.44 69.85) (xy 99.06 69.85)
-		)
-		(stroke
-			(width 0)
-			(type default)
-		)
-	)
-	(wire
-		(pts
 			(xy 92.71 129.54) (xy 96.52 129.54)
 		)
@@
 		)
 		(stroke
+			(width 0)
+			(type default)
+		)
+	)
+	(wire
+		(pts
+			(xy 97.79 71.12) (xy 91.44 71.12)
+		)
+		(stroke

Commit message: update
Other:
- title: Czujnik parametrów środowiskowych -> Enviromental parameters multi-sensor
Changed lines of the file:
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@@
 	(paper "A4")
 	(title_block
-		(title "Czujnik parametrów środowiskowych")
+		(title "Enviromental parameters multi-sensor")
 		(date "2026-01-20")
 		(rev "1.0")
